File: esp01flasher/esp01flasher.sch (KiCad schematic (older format))
At the start: 27 parts, among them J1 USB MiniB, J2 GPIO, J3 3V3, J4 VBUS, J5 3V3, J6 VBUS, SW1 Reset, SW2 Flash, U1 FT230XS, U2 AP2127N-3.3, U3 ESP-01

Commit message: PCB Layout
Parts:
- removed J3: 3V3, Connector_PinHeader_2.54mm:PinHeader_1x02_P2.54mm_Vertical, symbol Connector_Generic:Conn_01x02
- removed J6: VBUS, Connector_PinHeader_2.54mm:PinHeader_1x02_P2.54mm_Vertical, symbol Connector_Generic:Conn_01x02
- removed SW1: Reset, symbol Switch:SW_Push
- removed SW2: Flash, symbol Switch:SW_Push
- added SW1: Reset, tactile_switches:B3FS-1012P, symbol tactile_switches:B3FS-1012P
- added SW2: Flash, tactile_switches:B3FS-1012P, symbol tactile_switches:B3FS-1012P
- J1: value USB MiniB -> USB Mini B
- U3: value ESP-01 -> ESP-01v090
- renumbered D3 to D2, D2 to D3, J5 to J2, J4 to J3, J2 to J6, R2 to R1, R1 to R2, R7 to R4, R8 to R5, R4 to R6, R5 to R7, R6 to R8, U2 to U1, U1 to U2
Connections:
- net GND: now also SW1.3, SW2.3
- net at R6.2, U3.5 (RST): now also SW1.1
- net at J6.2 (Pin_2), R8.2, U3.6 (GPIO0): now also SW2.1
